Commit message: Add foot pin URDF and OBJ files; update ligament creation and simulation parameters
- Introduced a new URDF file for the foot pin model, defining its visual, collision, and inertial properties.
- Added the corresponding OBJ file for the foot pin geometry.
- Modified the ligament creation function to use the correct link index and adjusted the number of anchors.
- Updated the foot model in the simulation to use the new foot pin URDF, changing its mass and friction properties.
- Enhanced the constraint creation logic for the foot model, ensuring proper positioning and orientation.
- Adjusted simulation parameters, including the number of simulation steps and friction settings for better stability.
- Cleaned up commented-out code and added debug print statements for better traceability during simulation.

File: fracturesurgeryenv/gym_fracture/envs/Assets/241206/distal.urdf (robot description, URDF)
Before this commit: robot ., 1 links, 0 joints
Links:
- link _name: geometry collision mesh filename=./distal_rect_vhacd.obj scale=1 1 1; visual mesh filename=./distalrect.obj scale=1 1 1

File: fracturesurgeryenv/gym_fracture/envs/Assets/241206/distal1.urdf (robot description, URDF)
Before this commit: robot ., 1 links, 0 joints
Links:
- link _name: geometry collision mesh filename=./distal_rect.obj scale=1 1 1; visual mesh filename=./distal_rect.obj scale=1 1 1
