Commit message: - Changed dynamics - Updated force logging - Changed pin asset

File: fracturesurgeryenv/gym_fracture/envs/Assets/footpin.urdf (robot description, URDF)
Before this commit: robot ball_joint_object, 2 links, 1 joints
Links:
- link base_link: mass 1 -> 1.0; geometry collision mesh filename=./pin4.obj scale=1 1 1; visual mesh filename=pin4.obj scale=1 1 1

File: fracturesurgeryenv/gym_fracture/envs/Assets/legankle.urdf (robot description, URDF)
Before this commit: robot ball_joint_object, 2 links, 1 joints
Joints:
- joint yaw_joint: limit lower=-3.14 upper=3.14 effort=1.0 velocity=2.0 -> lower=-1.57 upper=1.57 effort=1.0 velocity=2.0

Commit message: - changed dynamics - changed position of the robot - changed the pin urdf

File: fracturesurgeryenv/gym_fracture/envs/Assets/footpin.urdf (robot description, URDF)
Before this commit: robot ball_joint_object, 2 links, 1 joints
Links:
- link base_link: mass 1.0 -> 1; geometry collision box size=0.008 0.01 0.08; visual box size=0.008 0.01 0.08
- link moving_link: geometry collision mesh filename=./anklenotibia_vhacd.obj scale=1 1 1; visual mesh filename=./anklenotibia.obj scale=1 1 1

File: fracturesurgeryenv/gym_fracture/envs/Assets/legankle.urdf (robot description, URDF)
Before this commit: robot ball_joint_object, 2 links, 1 joints
Links:
- link moving_link: geometry collision mesh filename=./proximal1_vhacd.obj scale=1 1 1; visual mesh filename=./proximal1.obj scale=1 1 1

Commit message: - test changes

File: fracturesurgeryenv/gym_fracture/envs/Assets/footpin.urdf (robot description, URDF)
Before this commit: robot ball_joint_object, 2 links, 1 joints
Links:
- link moving_link: geometry collision mesh filename=./foot4_vhacd.obj scale=1 1 1; visual mesh filename=./foot4.obj scale=1 1 1
Joints:
- joint yaw_joint: origin xyz=-0 0 0 rpy=-0 0 0 -> xyz=0.025 -0.04 0 rpy=0 1.57 0

File: fracturesurgeryenv/gym_fracture/envs/Assets/legankle.urdf (robot description, URDF)
Before this commit: robot ball_joint_object, 2 links, 1 joints
Links:
- removed link base_link
- link moving_link: geometry collision mesh filename=./leg_centre_vhacd.obj scale=1 1 1; visual mesh filename=./leg_centre.obj scale=1 1 1
Joints:
- removed joint yaw_joint

File: fracturesurgeryenv/gym_fracture/envs/Assets/legankle_orig.urdf (robot description, URDF)
Before this commit: robot ball_joint_object, 2 links, 1 joints
Joints:
- joint yaw_joint: origin xyz=0 0 0 rpy=0 0 0 -> xyz=0.02 0 0 rpy=0 0 1.57

Commit message: - changed to original urdf of 3d model

File: fracturesurgeryenv/gym_fracture/envs/Assets/footpin.urdf (robot description, URDF)
Before this commit: robot ball_joint_object, 2 links, 1 joints
Links:
- link moving_link: geometry collision mesh filename=./foot3_vhacd.obj scale=1 1 1; visual mesh filename=./foot3.obj scale=1 1 1
Joints:
- joint yaw_joint: origin xyz=-0 0 0 rpy=-0 0 0 -> xyz=0.03 -0.03 0 rpy=0 1.57 0
