Commit message: - removed force -fixed fouractions reward function

File: fracturesurgeryenv/gym_fracture/envs/Assets/legankle.urdf (robot description, URDF)
Before this commit: robot ball_joint_object, 2 links, 1 joints
Joints:
- joint yaw_joint: type fixed -> spherical

Commit message: - Final checks before testing

File: fracturesurgeryenv/gym_fracture/envs/Assets/legankle.urdf (robot description, URDF)
Before this commit: robot ball_joint_object, 2 links, 1 joints
Links:
- link moving_link: geometry collision mesh filename=./leg3_vhacd.obj scale=1 1 1; visual mesh filename=./leg3.obj scale=1 1 1
