Commit message: - Added new patient - Changed layout -Updated force (new_band) - Added force and contact to reward/done

File: fracturesurgeryenv/gym_fracture/envs/Assets/legankle_orig.urdf (robot description, URDF)
Before this commit: robot ball_joint_object, 2 links, 1 joints
Links:
- link base_link: mass 1 -> 0
Joints:
- joint yaw_joint: origin xyz=0.02 0 0 rpy=0 0 1.57 -> xyz=0.0 0 0 rpy=0 0 1.57
