Commit message: - testing different lig placement and more iterations

File: fracturesurgeryenv/gym_fracture/envs/Assets/Patient110/proximal.urdf (robot description, URDF)
Before this commit: robot proximal.obj, 2 links, 1 joints
Joints:
- joint leg: origin xyz=0.0009518 -0.0498613 0.4550867  rpy=0 0 0 -> xyz=0.0009518 -0.0498613 0.4550867 rpy=0 0 0
