Commit message: -updated dynamics - changed collision so the foot only collides with leg not soft tissue for stability

File: fracturesurgeryenv/gym_fracture/envs/Assets/Patient110/distal.urdf (robot description, URDF)
Before this commit: robot L_shaped_tool, 3 links, 2 joints
Links:
- link base_link: mass 0.0001 -> 0.01
- link moving_link: geometry collision mesh filename=distal_vhacd.obj scale=1 1 1; visual mesh filename=distal.obj scale=1 1 1
- link pin_link: mass 0.0001 -> 0.01

Commit message: Refine dynamics and observation handling in fracture surgery environment
- Reduced collision margin in foot dynamics to improve stability.
- Adjusted goal shape in observation space to account for new contact handling.
- Enabled goal cube creation for visual representation.
- Improved contact detection logic between foot and leg, ensuring accurate contact state.
- Modified goal position generation to use fixed extreme values for debugging.

File: fracturesurgeryenv/gym_fracture/envs/Assets/Patient110/distal.urdf (robot description, URDF)
Before this commit: robot L_shaped_tool, 3 links, 2 joints
Links:
- link moving_link: geometry collision mesh filename=decomp.obj scale=1 1 1; visual mesh filename=distal.obj scale=1 1 1

File: fracturesurgeryenv/gym_fracture/envs/Assets/Patient110/proximal.urdf (robot description, URDF)
Before this commit: robot proximal.obj, 2 links, 1 joints
Links:
- link proximal: geometry collision mesh filename=proximal_decomp.obj scale=1 1 1; visual mesh filename=proximal.obj scale=1 1 1
