Commit message: Refactor dynamics and environment setup in fracture surgery simulation
- Updated the import path for `change_ligament_dynamics` in `createligament.py`.
- Increased lateral friction and adjusted collision margin in `change_robot_dynamics`.
- Modified damping parameters in `change_ligament_dynamics` for improved simulation stability.
- Changed import path for `utils` in `env_utils.py`.
- Introduced a new parameter `patient` in `fracturesurgery_v2.py` to dynamically load patient-specific assets.
- Adjusted leg start positions and orientations based on patient type for better alignment.
- Updated finger force logic for soft tissue handling.
- Commented out goal configuration validation to prevent unnecessary checks during simulation.
- Enhanced young's modulus handling based on the environment type.

File: fracturesurgeryenv/gym_fracture/versions/v2/Assets/Patient110/distal.urdf (robot description, URDF)
Before this commit: robot L_shaped_tool, 3 links, 2 joints
Links:
- link moving_link: geometry collision mesh filename=decomp.obj scale=1 1 1; visual mesh filename=distal.obj scale=1 1 1
Joints:
- joint ankle_mount_joint: origin xyz=-0.0 0.02 -0.08 rpy=1.57 0 0 -> xyz=-0.0 -0.01 -0.08 rpy=1.57 0 0

File: fracturesurgeryenv/gym_fracture/versions/v2/Assets/Patient110/proximal.urdf (robot description, URDF)
Before this commit: robot proximal.obj, 2 links, 1 joints
Links:
- link proximal: geometry collision mesh filename=proximal_decomp.obj scale=1 1 1; visual mesh filename=proximal.obj scale=1 1 1
Joints:
- joint leg: origin xyz=0.0009518 -0.1498613 0.4550867 rpy=0 0 0 -> xyz=0.0009518 -0.0498613 0.4550867 rpy=0 0 0
