Commit message: test testing and none

File: fracturesurgeryenv/gym_fracture/versions/v2/Assets/Patient110/distal_copy.urdf (robot description, URDF)
Before this commit: robot L_shaped_tool, 3 links, 2 joints
Joints:
- joint ankle_mount_joint: origin xyz=0 0.08 -0.01 rpy=-1.57 0 0 -> xyz=0 0.08 0.03 rpy=-1.57 0 0

Commit message: just want to see if a smaller pin makes a difference

File: fracturesurgeryenv/gym_fracture/versions/v2/Assets/Patient110/distal_copy.urdf (robot description, URDF)
Before this commit: robot L_shaped_tool, 3 links, 2 joints
Links:
- link pin_link: geometry collision box size=0.008 0.01 0.08; visual box size=0.001 0.001 0.08

Commit message: collision too

File: fracturesurgeryenv/gym_fracture/versions/v2/Assets/Patient110/distal_copy.urdf (robot description, URDF)
Before this commit: robot L_shaped_tool, 3 links, 2 joints
Links:
- link pin_link: geometry collision box size=0.001 0.001 0.08; visual box size=0.001 0.001 0.08
