Commit message: this works for patient 252 -

File: fracturesurgeryenv/gym_fracture/versions/v2/Assets/Patient252/distal.urdf (robot description, URDF)
Before this commit: robot L_shaped_tool, 3 links, 2 joints
Links:
- link moving_link: geometry collision mesh filename=distal_252.obj scale=1 1 1; visual mesh filename=distal_252.obj scale=1 1 1
Joints:
- joint ankle_mount_joint: origin xyz=-0.0 0.01 -0.1 rpy=1.57 0 0 -> xyz=-0.0 -0.01 -0.08 rpy=1.57 0 0
