Commit message: kind of working for 102 - need to figure out why it can't quite get to goal

File: fracturesurgeryenv/gym_fracture/versions/v2/Assets/Patient102/distal.urdf (robot description, URDF)
Before this commit: robot L_shaped_tool, 3 links, 2 joints
Links:
- link moving_link: geometry collision mesh filename=distal1022_vhacd.obj scale=1 1 1; visual mesh filename=distal102.obj scale=1 1 1

File: fracturesurgeryenv/gym_fracture/versions/v2/Assets/Patient102/proximal.urdf (robot description, URDF)
Before this commit: robot proximal.obj, 2 links, 1 joints
Links:
- link proximal: geometry collision mesh filename=proximal1022_vhacd.obj scale=1 1 1; visual mesh filename=proximal_102.obj scale=1 1 1
