Commit message: - V2 for testing - Main changes involve changing the distal bone to be the base rather than the pin

File: fracturesurgeryenv/gym_fracture/versions/v2/Assets/Patient102/proximal.urdf (robot description, URDF)
Before this commit: robot proximal.obj, 2 links, 1 joints
Links:
- link proximal: geometry collision mesh filename=proximal1022_vhacd.obj scale=0.95 0.95 0.95; visual mesh filename=proximal_102.obj scale=1 1 1

File: fracturesurgeryenv/gym_fracture/versions/v2/Assets/Patient126/proximal.urdf (robot description, URDF)
Before this commit: robot proximal_126.obj, 2 links, 1 joints
Links:
- link proximal_126: geometry collision mesh filename=proximal_1262_vhacd.obj scale=0.9 0.9 0.9; visual mesh filename=proximal_1262.obj scale=1 1 1

File: fracturesurgeryenv/gym_fracture/versions/v2/Assets/Patient252/distal.urdf (robot description, URDF)
Before this commit: robot L_shaped_tool, 3 links, 2 joints
Links:
- link moving_link: geometry collision mesh filename=distal_252.obj scale=0.9 0.9 0.9; visual mesh filename=distal_252.obj scale=1 1 1

File: fracturesurgeryenv/gym_fracture/versions/v2/Assets/Patient252/proximal.urdf (robot description, URDF)
Before this commit: robot proximal.obj, 2 links, 1 joints
Links:
- link proximal: geometry collision mesh filename=proximal_252_vhacd.obj scale=0.9 0.9 0.9; visual mesh filename=proximal_2522.obj scale=1 1 1
