Commit message: this works for patient 198

File: fracturesurgeryenv/gym_fracture/versions/v2/Assets/Patient198/distal.urdf (robot description, URDF)
Before this commit: robot distal.obj, 3 links, 2 joints
Links:
- link moving_link: geometry collision mesh filename=distal_198_vhacd.obj scale=0.9 0.9 0.9; visual mesh filename=distal_198.obj scale=1 1 1

File: fracturesurgeryenv/gym_fracture/versions/v2/Assets/Patient198/proximal.urdf (robot description, URDF)
Before this commit: robot proximal_126.obj, 2 links, 1 joints
Links:
- link proximal_126: geometry collision mesh filename=proximal_198_vhacd.obj scale=0.9 0.9 0.9; visual mesh filename=proximal_198.obj scale=1 1 1
