Commit message: new proximal was in wrong place

File: fracturesurgeryenv/gym_fracture/versions/v2/Assets/Patient198/proximal.urdf (robot description, URDF)
Before this commit: robot proximal_126.obj, 2 links, 1 joints
Links:
- link proximal_126: geometry collision mesh filename=proximal_19822_vhacd.obj scale=1 1 1; visual mesh filename=proximal_198.obj scale=1 1 1
