Commit message: patient 132 works here note, made the fragment weigh less due to much smaller piece

File: fracturesurgeryenv/gym_fracture/versions/v2/Assets/Patient132/distal.urdf (robot description, URDF)
Before this commit: robot distal_132.obj, 3 links, 2 joints
Links:
- link moving_link: geometry collision mesh filename=distal_132_vhacd.obj scale=1 1 1; visual mesh filename=distal1322.obj scale=1 1 1

File: fracturesurgeryenv/gym_fracture/versions/v2/Assets/Patient132/proximal.urdf (robot description, URDF)
Before this commit: robot proximal_132.obj, 2 links, 1 joints
Links:
- link proximal_132: geometry collision mesh filename=proximal_132_vhacd.obj scale=1 1 1; visual mesh filename=proximal132.obj scale=1 1 1
Joints:
- joint leg: origin xyz=0.0009518 -0.5498613 0.04550867 rpy=0 0 0 -> xyz=0.0109518 -0.4898613 -0.051850867 rpy=1.57 0 0
