Commit message: v1 ready for sweep

File: fracturesurgeryenv/gym_fracture/versions/v1/Assets/Patient110/distal.urdf (robot description, URDF)
Before this commit: robot L_shaped_tool, 3 links, 2 joints
Joints:
- joint ankle_mount_joint: origin xyz=-0.0 0.02 -0.08 rpy=1.57 0 0 -> xyz=-0.0 -0.01 -0.08 rpy=1.57 0 0

Commit message: just saving work up to here, atm this all works (well not the contact thing)

File: fracturesurgeryenv/gym_fracture/versions/v1/Assets/Patient110/distal.urdf (robot description, URDF)
Before this commit: robot L_shaped_tool, 3 links, 2 joints
Joints:
- joint ankle_mount_joint: origin xyz=-0.0 -0.01 -0.08 rpy=1.57 0 0 -> xyz=-0.0 0.03 -0.08 rpy=1.57 0 0

File: fracturesurgeryenv/gym_fracture/versions/v2/Assets/Patient102/distal_copy.urdf (robot description, URDF)
Before this commit: robot L_shaped_tool, 3 links, 2 joints
Joints:
- joint ankle_mount_joint: origin xyz=0 0.08 -0.01 rpy=-1.57 0 0 -> xyz=0 0.08 0.03 rpy=-1.57 0 0

File: fracturesurgeryenv/gym_fracture/versions/v2/Assets/Patient126/distal_copy.urdf (robot description, URDF)
Before this commit: robot L_shaped_tool, 3 links, 2 joints
Joints:
- joint ankle_mount_joint: origin xyz=0 0.08 0.002 rpy=-1.57 0 0 -> xyz=0 0.08 0.0 rpy=-1.57 0 0

File: fracturesurgeryenv/gym_fracture/versions/v2/Assets/Patient198/distal_copy.urdf (robot description, URDF)
Before this commit: robot L_shaped_tool, 3 links, 2 joints
Joints:
- joint ankle_mount_joint: origin xyz=0 0.0 0.08 rpy=0 0 0 -> xyz=0 -0.03 0.08 rpy=0 0 0

File: fracturesurgeryenv/gym_fracture/versions/v2/Assets/Patient252/distal_copy.urdf (robot description, URDF)
Before this commit: robot L_shaped_tool, 3 links, 2 joints
Joints:
- joint ankle_mount_joint: origin xyz=0 0.08 -0.01 rpy=-1.57 0 0 -> xyz=0 0.08 0.03 rpy=-1.57 0 0
