Commit message: ready for patient testing

File: fracturesurgeryenv/gym_fracture/versions/v2/Assets/Patient126/distal_copy.urdf (robot description, URDF)
Before this commit: robot L_shaped_tool, 3 links, 2 joints
Links:
- link pin_link: geometry collision box size=0.001 0.001 0.08; visual box size=0.001 0.001 0.08

File: fracturesurgeryenv/gym_fracture/versions/v2/Assets/Patient132/distal_copy.urdf (robot description, URDF)
Before this commit: robot L_shaped_tool, 3 links, 2 joints
Links:
- link pin_link: geometry collision box size=0.001 0.001 0.08; visual box size=0.001 0.001 0.08

File: fracturesurgeryenv/gym_fracture/versions/v2/Assets/Patient132/proximal.urdf (robot description, URDF)
Before this commit: robot proximal_132.obj, 2 links, 1 joints
Links:
- link proximal_132: geometry collision mesh filename=proximal_132_vhacd.obj scale=0.9 0.9 0.9; visual mesh filename=proximal132.obj scale=1 1 1

File: fracturesurgeryenv/gym_fracture/versions/v2/Assets/Patient198/distal_copy.urdf (robot description, URDF)
Before this commit: robot L_shaped_tool, 3 links, 2 joints
Links:
- link pin_link: geometry collision box size=0.001 0.001 0.08; visual box size=0.001 0.001 0.08

File: fracturesurgeryenv/gym_fracture/versions/v2/Assets/Patient198/proximal.urdf (robot description, URDF)
Before this commit: robot proximal_126.obj, 2 links, 1 joints
Links:
- link proximal_126: geometry collision mesh filename=proximal_1982_vhacd.obj scale=1 1 1; visual mesh filename=proximal_198.obj scale=1 1 1
